Commit message: node to convert imu magnetometor data to azimuth in angles

File: urdf/husky.urdf.xacro (robot description, xacro)
@@ -53,5 +53,5 @@
   <xacro:arg name="laser_ust10_rear_rpy"      default="$(optenv HUSKY_UST10_SECONDARY_RPY 0 0 3.14159)" />
   <!-- Velodyne LiDAR Primary and Secondary -->
-  <xacro:arg name="laser_3d_enabled"              default="$(optenv HUSKY_LASER_3D_ENABLED 0)" />
+  <xacro:arg name="laser_3d_enabled"              default="$(optenv HUSKY_LASER_3D_ENABLED 1)" />
   <xacro:arg name="laser_3d_topic"                default="$(optenv HUSKY_LASER_3D_TOPIC points)"/>
   <xacro:arg name="laser_3d_tower"                default="$(optenv HUSKY_LASER_3D_TOWER 1)"/>
@@ -68,5 +68,5 @@
   <xacro:arg name="laser_3d_secondary_rpy"        default="$(optenv HUSKY_LASER_3D_SECONDARY_RPY 0 0 -3.14159)" />
   <!-- Realsense Camera Primary and Secondary -->
-  <xacro:arg name="realsense_enabled"             default="$(optenv HUSKY_REALSENSE_ENABLED 0)" />
+  <xacro:arg name="realsense_enabled"             default="$(optenv HUSKY_REALSENSE_ENABLED 1)" />
   <xacro:arg name="realsense_topic"               default="$(optenv HUSKY_REALSENSE_TOPIC realsense)" />
   <xacro:arg name="realsense_prefix"              default="$(optenv HUSKY_REALSENSE_PREFIX camera)" />
@@ -113,5 +113,5 @@
   <xacro:include filename="$(find husky_description)/urdf/accessories/sensor_arch.urdf.xacro"/>
   <xacro:include filename="$(find husky_description)/urdf/accessories/sick_lms1xx_mount.urdf.xacro"/>
-  <xacro:include filename="$(find husky_description)/urdf/accessories/vlp16_mount.urdf.xacro"/>
+<!--  <xacro:include filename="$(find husky_description)/urdf/accessories/vlp16_mount.urdf.xacro"/>-->
   <xacro:include filename="$(find husky_description)/urdf/decorations.urdf.xacro" />
   <xacro:include filename="$(find husky_description)/urdf/wheel.urdf.xacro" />
@@ -290,30 +290,4 @@
 <!--    </xacro:unless>-->
 <!--  </xacro:if>-->
-  <!-- Ouster sensor links and fixed joints -->
-    <joint name="ouster_base_mount_joint" type="fixed">
-      <origin xyz="$(arg laser_3d_xyz)" rpy="$(arg laser_3d_rpy)" />
-      <parent link="$(arg laser_3d_parent)"/>
-      <child link="ouster_link"/>
-    </joint>
-    <link name="ouster_link">
-      <inertial>
-         <mass value="0.33"/>
-         <origin xyz="0 0 0.0365" rpy="0 0 0" />
-         <inertia ixx="0.000241148" ixy="0" ixz="0"
-          iyy="0.000241148" iyz="0" izz="0.000264"/>
-      </inertial>
-      <collision name="base_collision">
-         <origin xyz="0 0 0.0365" rpy="0 0 0" />
-         <geometry>
- 	   <cylinder radius="0.04" length="0.073"/>
-         </geometry>
-      </collision>
-      <visual name="base_visual">
-         <origin xyz="0 0 0" rpy="0 0 1.5707" />
-         <geometry>
-	    <mesh filename="package://ouster_description/meshes/os1_64.dae" />
-         </geometry>
-      </visual>
-   </link>
   <gazebo>
     <plugin name="gazebo_ros_control" filename="libgazebo_ros_control.so">
@@ -342,6 +316,6 @@
       <bodyName>base_link</bodyName>
       <frameId>base_link</frameId>
-      <topicName>navsat/fix</topicName>
-      <velocityTopicName>navsat/vel</velocityTopicName>
+      <topicName>/fix</topicName>
+      <velocityTopicName>/vel</velocityTopicName>
       <referenceLatitude>49.9</referenceLatitude>
       <referenceLongitude>8.9</referenceLongitude>
@@ -351,8 +325,34 @@
     </plugin>
   </gazebo>
-  <!-- Gazebo requires the ouster_gazebo_plugins package -->
-    <gazebo reference="ouster_link">
+  <xacro:if value="$(arg laser_3d_enabled)">
+    <!-- Ouster sensor links and fixed joints -->
+    <joint name="ouster_base_mount_joint" type="fixed">
+      <origin xyz="$(arg laser_3d_xyz)" rpy="$(arg laser_3d_rpy)" />
+      <parent link="$(arg laser_3d_parent)"/>
+      <child link="ouster_link"/>
+    </joint>
+    <link name="ouster_link">
+      <inertial>
+         <mass value="0.33"/>
+         <origin xyz="0 0 0.0365" rpy="0 0 0" />
+         <inertia ixx="0.000241148" ixy="0" ixz="0"
+          iyy="0.000241148" iyz="0" izz="0.000264"/>
+      </inertial>
+      <collision name="base_collision">
+         <origin xyz="0 0 0.0365" rpy="0 0 0" />
+         <geometry>
+ 	   <cylinder radius="0.04" length="0.073"/>
+         </geometry>
+      </collision>
+      <visual name="base_visual">
+         <origin xyz="0 0 0" rpy="0 0 1.5707" />
+         <geometry>
+	    <mesh filename="package://ouster_description/meshes/os1_64.dae" />
+         </geometry>
+      </visual>
+    </link>
+    <!-- Gazebo requires the ouster_gazebo_plugins package -->
+    <gazebo eference="ouster_link">
         <sensor type="ray" name="ouster-OS1-64">
-<!--          <pose>0 0 0 0 0 0</pose>-->
           <pose>0 0 0.035925 0 0 0</pose>
           <visualize>false</visualize>
@@ -362,5 +362,4 @@
             <scan>
               <horizontal>
-<!--                <samples>220</samples>-->
                 <samples>1024</samples>
                 <resolution>1</resolution>
@@ -369,9 +368,6 @@
               </horizontal>
               <vertical>
-<!--                <samples>64</samples>-->
                 <samples>128</samples>
 		        <resolution>1</resolution>
-<!--                <min_angle>-0.26</min_angle> &lt;!&ndash;15*3.1415926535897931/180.0&ndash;&gt;-->
-<!--                <max_angle>0.26</max_angle>-->
                 <min_angle>-${pi/4}</min_angle>
                 <max_angle>${pi/4}</max_angle>
@@ -379,7 +375,4 @@
             </scan>
             <range>
-<!--              <min>0.9</min>-->
-<!--              <max>75</max>-->
-<!--              <resolution>0.03</resolution>-->
               <min>0.25</min>  <!-- Datasheet says 0 cm, but that's a lie. -->
               <max>50</max>
@@ -389,5 +382,4 @@
               <type>gaussian</type>
               <mean>0.0</mean>
-<!--              <stddev>0.0</stddev>-->
               <stddev>0.01</stddev>
             </noise>
@@ -402,4 +394,5 @@
         </sensor>
     </gazebo>
+  </xacro:if>
   <!-- Optional custom includes. -->
   <xacro:include filename="$(arg urdf_extras)" />

Commit message: created simple gpx file for simulator and added path follower node call

File: urdf/husky.urdf.xacro (robot description, xacro)
@@ -53,5 +53,5 @@
   <xacro:arg name="laser_ust10_rear_rpy"      default="$(optenv HUSKY_UST10_SECONDARY_RPY 0 0 3.14159)" />
   <!-- Velodyne LiDAR Primary and Secondary -->
-  <xacro:arg name="laser_3d_enabled"              default="$(optenv HUSKY_LASER_3D_ENABLED 1)" />
+  <xacro:arg name="laser_3d_enabled"              default="$(optenv HUSKY_LASER_3D_ENABLED 0)" />
   <xacro:arg name="laser_3d_topic"                default="$(optenv HUSKY_LASER_3D_TOPIC points)"/>
   <xacro:arg name="laser_3d_tower"                default="$(optenv HUSKY_LASER_3D_TOWER 1)"/>
@@ -68,5 +68,5 @@
   <xacro:arg name="laser_3d_secondary_rpy"        default="$(optenv HUSKY_LASER_3D_SECONDARY_RPY 0 0 -3.14159)" />
   <!-- Realsense Camera Primary and Secondary -->
-  <xacro:arg name="realsense_enabled"             default="$(optenv HUSKY_REALSENSE_ENABLED 1)" />
+  <xacro:arg name="realsense_enabled"             default="$(optenv HUSKY_REALSENSE_ENABLED 0)" />
   <xacro:arg name="realsense_topic"               default="$(optenv HUSKY_REALSENSE_TOPIC realsense)" />
   <xacro:arg name="realsense_prefix"              default="$(optenv HUSKY_REALSENSE_PREFIX camera)" />
@@ -342,5 +342,5 @@
          <origin xyz="0 0 0.0365" rpy="0 0 0" />
          <geometry>
- 	   <cylinder radius="0.04" length="0.073"/>
+       <cylinder radius="0.04" length="0.073"/>
          </geometry>
       </collision>
@@ -348,49 +348,49 @@
          <origin xyz="0 0 0" rpy="0 0 1.5707" />
          <geometry>
-	    <mesh filename="package://ouster_description/meshes/os1_64.dae" />
+        <mesh filename="package://ouster_description/meshes/os1_64.dae" />
          </geometry>
       </visual>
     </link>
     <!-- Gazebo requires the ouster_gazebo_plugins package -->
-    <gazebo eference="ouster_link">
-        <sensor type="ray" name="ouster-OS1-64">
-          <pose>0 0 0.035925 0 0 0</pose>
-          <visualize>false</visualize>
-          <update_rate>10</update_rate>
-          <always_on>1</always_on>
-          <ray>
-            <scan>
-              <horizontal>
-                <samples>1024</samples>
-                <resolution>1</resolution>
-                <min_angle>-3.1415926535897931</min_angle>
-                <max_angle>3.1415926535897931</max_angle>
-              </horizontal>
-              <vertical>
-                <samples>128</samples>
-		        <resolution>1</resolution>
-                <min_angle>-${pi/4}</min_angle>
-                <max_angle>${pi/4}</max_angle>
-              </vertical>
-            </scan>
-            <range>
-              <min>0.25</min>  <!-- Datasheet says 0 cm, but that's a lie. -->
-              <max>50</max>
-              <resolution>0.01</resolution>
-            </range>
-            <noise>
-              <type>gaussian</type>
-              <mean>0.0</mean>
-              <stddev>0.01</stddev>
-            </noise>
-          </ray>
-          <plugin name="gazebo_ros_laser_controller" filename="libgazebo_ros_ouster_laser.so">
-            <topicName>/points</topicName>
-            <frameName>ouster_link</frameName>
-            <min_range>0.9</min_range>
-            <max_range>75</max_range>
-            <gaussianNoise>0.008</gaussianNoise>
-          </plugin>
-        </sensor>
+    <gazebo reference="ouster_link">
+      <sensor type="ray" name="ouster-OS1-64">
+        <pose>0 0 0.035925 0 0 0</pose>
+        <visualize>false</visualize>
+        <update_rate>10</update_rate>
+        <always_on>1</always_on>
+        <ray>
+          <scan>
+            <horizontal>
+              <samples>1024</samples>
+              <resolution>1</resolution>
+              <min_angle>-3.1415926535897931</min_angle>
+              <max_angle>3.1415926535897931</max_angle>
+            </horizontal>
+            <vertical>
+              <samples>128</samples>
+              <resolution>1</resolution>
+              <min_angle>-${pi/4}</min_angle>
+              <max_angle>${pi/4}</max_angle>
+            </vertical>
+          </scan>
+          <range>
+            <min>0.25</min>  <!-- Datasheet says 0 cm, but that's a lie. -->
+            <max>50</max>
+            <resolution>0.01</resolution>
+          </range>
+          <noise>
+            <type>gaussian</type>
+            <mean>0.0</mean>
+            <stddev>0.01</stddev>
+          </noise>
+        </ray>
+        <plugin name="gazebo_ros_laser_controller" filename="libgazebo_ros_ouster_laser.so">
+          <topicName>/points</topicName>
+          <frameName>ouster_link</frameName>
+          <min_range>0.9</min_range>
+          <max_range>75</max_range>
+          <gaussianNoise>0.008</gaussianNoise>
+        </plugin>
+      </sensor>
     </gazebo>
   </xacro:if>

Commit message: using gpu to render ouster lidar cloud

File: urdf/husky.urdf.xacro (robot description, xacro)
@@ -107,4 +107,6 @@
   <xacro:arg name="urdf_extras"     default="$(optenv HUSKY_URDF_EXTRAS empty.urdf)" />
   <xacro:arg name="cpr_urdf_extras" default="$(optenv CPR_URDF_EXTRAS empty.urdf)" />
+<!--  <xacro:arg name="gpu" default="true"/>-->
+<!--  <xacro:property name="gpu" value="$(arg gpu)" />-->
   <!-- Included URDF/XACRO Files -->
   <xacro:include filename="$(find husky_description)/urdf/accessories/hokuyo_ust10.urdf.xacro" />
@@ -403,5 +405,6 @@
           </noise>
         </ray>
-        <plugin name="gazebo_ros_laser_controller" filename="libgazebo_ros_ouster_laser.so">
+<!--        <plugin name="gazebo_ros_laser_controller" filename="libgazebo_ros_ouster_laser.so">-->
+        <plugin name="gazebo_ros_laser_controller" filename="libgazebo_ros_ouster_gpu_laser.so">
           <topicName>/points</topicName>
           <frameName>ouster_link</frameName>

Commit message: fov vis, control path vis, gps link in urdf file

File: urdf/husky.urdf.xacro (robot description, xacro)
@@ -312,4 +312,10 @@
     </plugin>
   </gazebo>
+  <joint name="gps_base_mount_joint" type="fixed">
+    <origin xyz="0 0 0" rpy="0 0 0" />
+    <parent link="base_link"/>
+    <child link="gps"/>
+  </joint>
+  <link name="gps"/>
   <gazebo>
     <plugin name="gps_controller" filename="libhector_gazebo_ros_gps.so">
@@ -373,6 +379,8 @@
     </link>
     <!-- Gazebo requires the ouster_gazebo_plugins package -->
+    <!-- Run Ouster plugin with GPU: https://engcang.github.io/Ouster-Gazebo-Plugin-boosting-up-with-GPU-ray/ -->
     <gazebo reference="ouster_link">
-      <sensor type="ray" name="ouster-OS1-64">
+<!--      <sensor type="ray" name="ouster-OS1-64">-->
+      <sensor type="gpu_ray" name="ouster-OS1-64">
         <pose>0 0 0.035925 0 0 0</pose>
         <visualize>false</visualize>

Commit message: Update realsense xacro

File: urdf/husky.urdf.xacro (robot description, xacro)
@@ -69,4 +69,5 @@
   <!-- Realsense Camera Primary and Secondary -->
   <xacro:arg name="realsense_enabled"             default="$(optenv HUSKY_REALSENSE_ENABLED 1)" />
+  <xacro:arg name="realsense_model"               default="$(optenv HUSKY_REALSENSE_MODEL d435)"/>
   <xacro:arg name="realsense_topic"               default="$(optenv HUSKY_REALSENSE_TOPIC realsense)" />
   <xacro:arg name="realsense_prefix"              default="$(optenv HUSKY_REALSENSE_PREFIX camera)" />
@@ -74,5 +75,7 @@
   <xacro:arg name="realsense_xyz"                 default="$(optenv HUSKY_REALSENSE_XYZ 0 0 0)" />
   <xacro:arg name="realsense_rpy"                 default="$(optenv HUSKY_REALSENSE_RPY 0 0 0)" />
+  <xacro:property name="realsense_model"          value="$(arg realsense_model)"/>
   <xacro:arg name="realsense_secondary_enabled"   default="$(optenv HUSKY_REALSENSE_SECONDARY_ENABLED 0)" />
+  <xacro:arg name="realsense_secondary_model"     default="$(optenv HUSKY_REALSENSE_SECONDARY_MODEL d435)"/>
   <xacro:arg name="realsense_secondary_topic"     default="$(optenv HUSKY_REALSENSE_SECONDARY_TOPIC realsense_secondary)" />
   <xacro:arg name="realsense_secondary_prefix"    default="$(optenv HUSKY_REALSENSE_SECONDARY_PREFIX camera_secondary)" />
@@ -80,4 +83,5 @@
   <xacro:arg name="realsense_secondary_xyz"       default="$(optenv HUSKY_REALSENSE_SECONDARY_XYZ 0 0 0)" />
   <xacro:arg name="realsense_secondary_rpy"       default="$(optenv HUSKY_REALSENSE_SECONDARY_RPY 0 0 0)" />
+  <xacro:property name="realsense_secondary_model" value="$(arg realsense_secondary_model)"/>
   <!-- BlackflyS Camera Primary and Secondary -->
   <xacro:arg name="blackfly_enabled"                  default="$(optenv HUSKY_BLACKFLY 0)"/>
@@ -242,21 +246,33 @@
   </xacro:if>
   <!-- Intel Realsense Primary and Secondary -->
+  <xacro:if value="${realsense_model == 'd435'}">
+    <xacro:include filename="$(find realsense2_description)/urdf/_d435.urdf.xacro" />
+  </xacro:if>
+  <xacro:if value="${realsense_model == 'd435i'}">
+    <xacro:include filename="$(find realsense2_description)/urdf/_d435i.urdf.xacro" />
+  </xacro:if>
+  <xacro:if value="${realsense_model == 'd415'}">
+    <xacro:include filename="$(find realsense2_description)/urdf/_d415.urdf.xacro" />
+  </xacro:if>
+  <xacro:if value="${realsense_model == 'd455'}">
+    <xacro:include filename="$(find realsense2_description)/urdf/_d435.urdf.xacro" />
+  </xacro:if>
   <xacro:if value="$(arg realsense_enabled)">
-    <link name="$(arg realsense_prefix)_realsense_mountpoint"/>
-    <joint name="$(arg realsense_prefix)_realsense_mountpoint_joint" type="fixed">
-      <origin xyz="$(arg realsense_xyz)" rpy="$(arg realsense_rpy)" />
-      <parent link="$(arg realsense_parent)"/>
-      <child link="$(arg realsense_prefix)_realsense_mountpoint" />
-    </joint>
-    <xacro:intel_realsense_mount prefix="$(arg realsense_prefix)" topic="$(arg realsense_topic)" parent_link="$(arg realsense_prefix)_realsense_mountpoint"/>
+    <xacro:realsense_sensor rs_model="$(arg realsense_model)"
+                            prefix="$(arg realsense_prefix)"
+                            parent="$(arg realsense_parent)"
+                            topic="$(arg realsense_topic)"
+                            include="0">
+      <origin xyz="$(arg realsense_xyz)" rpy="$(arg realsense_rpy)"/>
+    </xacro:realsense_sensor>
   </xacro:if>
   <xacro:if value="$(arg realsense_secondary_enabled)">
-    <link name="$(arg realsense_secondary_prefix)_realsense_mountpoint"/>
-    <joint name="$(arg realsense_secondary_prefix)_realsense_mountpoint_joint" type="fixed">
-      <origin xyz="$(arg realsense_secondary_xyz)" rpy="$(arg realsense_secondary_rpy)" />
-      <parent link="$(arg realsense_secondary_parent)"/>
-      <child link="$(arg realsense_secondary_prefix)_realsense_mountpoint" />
-    </joint>
-    <xacro:intel_realsense_mount prefix="$(arg realsense_secondary_prefix)" topic="$(arg realsense_secondary_topic)" parent_link="$(arg realsense_secondary_prefix)_realsense_mountpoint"/>
+    <xacro:realsense_sensor rs_model="$(arg realsense_secondary_model)"
+                            prefix="$(arg realsense_secondary_prefix)"
+                            parent="$(arg realsense_secondary_parent)"
+                            topic="$(arg realsense_secondary_topic)"
+                            include="0">
+      <origin xyz="$(arg realsense_secondary_xyz)" rpy="$(arg realsense_secondary_rpy)"/>
+    </xacro:realsense_sensor>
   </xacro:if>
   <!-- BlackflyS Camera Primary and Secondary -->

Commit message: standart (blackfly) camera instead of realsence

File: urdf/husky.urdf.xacro (robot description, xacro)
@@ -68,5 +68,5 @@
   <xacro:arg name="laser_3d_secondary_rpy"        default="$(optenv HUSKY_LASER_3D_SECONDARY_RPY 0 0 -3.14159)" />
   <!-- Realsense Camera Primary and Secondary -->
-  <xacro:arg name="realsense_enabled"             default="$(optenv HUSKY_REALSENSE_ENABLED 1)" />
+  <xacro:arg name="realsense_enabled"             default="$(optenv HUSKY_REALSENSE_ENABLED 0)" />
   <xacro:arg name="realsense_model"               default="$(optenv HUSKY_REALSENSE_MODEL d435)"/>
   <xacro:arg name="realsense_topic"               default="$(optenv HUSKY_REALSENSE_TOPIC realsense)" />
@@ -85,6 +85,6 @@
   <xacro:property name="realsense_secondary_model" value="$(arg realsense_secondary_model)"/>
   <!-- BlackflyS Camera Primary and Secondary -->
-  <xacro:arg name="blackfly_enabled"                  default="$(optenv HUSKY_BLACKFLY 0)"/>
-  <xacro:arg name="blackfly_mount_enabled"            default="$(optenv HUSKY_BLACKFLY_MOUNT_ENABLED 1)"/>
+  <xacro:arg name="blackfly_enabled"                  default="$(optenv HUSKY_BLACKFLY 1)"/>
+  <xacro:arg name="blackfly_mount_enabled"            default="$(optenv HUSKY_BLACKFLY_MOUNT_ENABLED 0)"/>
   <xacro:arg name="blackfly_mount_angle"              default="$(optenv HUSKY_BLACKFLY_MOUNT_ANGLE 0)"/>
   <xacro:arg name="blackfly_prefix"                   default="$(optenv HUSKY_BLACKFLY_PREFIX blackfly)"/>
@@ -93,5 +93,5 @@
   <xacro:arg name="blackfly_rpy"                      default="$(optenv HUSKY_BLACKFLY_RPY 0 0 0)"/>
   <xacro:arg name="blackfly_secondary_enabled"        default="$(optenv HUSKY_BLACKFLY_SECONDARY 0)"/>
-  <xacro:arg name="blackfly_secondary_mount_enabled"  default="$(optenv HUSKY_BLACKFLY_SECONDARY_MOUNT_ENABLED 1)"/>
+  <xacro:arg name="blackfly_secondary_mount_enabled"  default="$(optenv HUSKY_BLACKFLY_SECONDARY_MOUNT_ENABLED 0)"/>
   <xacro:arg name="blackfly_secondary_mount_angle"    default="$(optenv HUSKY_BLACKFLY_SECONDARY_MOUNT_ANGLE 0)"/>
   <xacro:arg name="blackfly_secondary_prefix"         default="$(optenv HUSKY_BLACKFLY_SECONDARY_PREFIX blackfly_secondary)"/>
@@ -296,16 +296,16 @@
     Velodyne 3D LiDAR Primary and Secondary
   -->
-<!--  <xacro:if value="$(arg laser_3d_enabled)">-->
-<!--    <xacro:if value="$(arg laser_3d_tower)">-->
-<!--      <xacro:vlp16_mount prefix="$(arg laser_3d_prefix)" parent_link="$(arg laser_3d_parent)" topic="$(arg laser_3d_topic)">-->
-<!--        <origin xyz="$(arg laser_3d_xyz)" rpy="$(arg laser_3d_rpy)" />-->
-<!--      </xacro:vlp16_mount>-->
-<!--    </xacro:if>-->
-<!--    <xacro:unless value="$(arg laser_3d_tower)">-->
-<!--      <xacro:VLP-16 parent="$(arg laser_3d_parent)" topic="$(arg laser_3d_topic)" name="$(arg laser_3d_prefix)velodyne">-->
-<!--        <origin xyz="$(arg laser_3d_xyz)" rpy="$(arg laser_3d_rpy)" />-->
-<!--      </xacro:VLP-16>-->
-<!--    </xacro:unless>-->
-<!--  </xacro:if>-->
+  <xacro:if value="$(arg laser_3d_secondary_enabled)">
+    <xacro:if value="$(arg laser_3d_tower)">
+      <xacro:vlp16_mount prefix="$(arg laser_3d_prefix)" parent_link="$(arg laser_3d_parent)" topic="$(arg laser_3d_topic)">
+        <origin xyz="$(arg laser_3d_xyz)" rpy="$(arg laser_3d_rpy)" />
+      </xacro:vlp16_mount>
+    </xacro:if>
+    <xacro:unless value="$(arg laser_3d_tower)">
+      <xacro:VLP-16 parent="$(arg laser_3d_parent)" topic="$(arg laser_3d_topic)" name="$(arg laser_3d_prefix)velodyne">
+        <origin xyz="$(arg laser_3d_xyz)" rpy="$(arg laser_3d_rpy)" />
+      </xacro:VLP-16>
+    </xacro:unless>
+  </xacro:if>
   <gazebo>
     <plugin name="gazebo_ros_control" filename="libgazebo_ros_control.so">
@@ -342,6 +342,4 @@
       <topicName>gps/fix</topicName>
       <velocityTopicName>/vel</velocityTopicName>
-<!--      <referenceLatitude>49.9</referenceLatitude>-->
-<!--      <referenceLongitude>8.9</referenceLongitude>-->
       <referenceLatitude>50.090337</referenceLatitude>
       <referenceLongitude>14.133275</referenceLongitude>
